File: rgb_mosfet_panel.kicad_pcb (KiCad board)
At the start: 2 copper layers, 80 x 79.5 mm, 89 parts, among them J1 USB_B_Micro, Q1 DMG2302U, Q2 DMG2302U, Q3 DMG2302U, Q4 DMG2302U, Q5 DMG2302U, U1 TC2014-3.3VxCTTR, U2 MCP1640CH, U3 ATtiny13A-SSU, X1 SXO-53C3A071

Commit message: Add ISP header
Parts:
- added J2: AVR-ISP-6, Connector_PinHeader_2.54mm:PinHeader_2x03_P2.54mm_Vertical_SMD, B.Cu at (72.1, 84.3)
Connections:
- net Net-(R8-Pad1) renamed RESET
- net R renamed MOSI
Routing:
- net RESET: track 0.00 -> 38.6 mm, vias 1 -> 4
- net B: track 2.67 -> 41.1 mm, vias 0 -> 4
- net G: track 2.36 -> 31.7 mm, vias 0 -> 4
- net +5V: track 96.0 -> 123.9 mm
- net MOSI: track 2.51 -> 27.1 mm, vias 0 -> 2
- net GND: vias 79 -> 81
