File: rgb_mosfet_panel.kicad_pcb (KiCad board)
At the start: 2 copper layers, 80 x 79.5 mm, 90 parts, among them J1 USB_B_Micro, J2 AVR-ISP-6, Q1 DMG2302U, Q2 DMG2302U, Q3 DMG2302U, Q4 DMG2302U, Q5 DMG2302U, U1 TC2014-3.3VxCTTR, U2 MCP1640CH, U3 ATtiny13A-SSU, X1 SXO-53C3A071

Commit message: Move around boost to hopefully work
Parts:
- added +12V: Test_Point_2.67x1.02mm, digikey-footprints:Test_Point_2.67x1.02mm, B.Cu at (100.9, 91.8)
- added GND: Test_Point_2.67x1.02mm, digikey-footprints:Test_Point_2.67x1.02mm, F.Cu at (106.3, 65.6)
- added VFB: Test_Point_2.67x1.02mm, digikey-footprints:Test_Point_2.67x1.02mm, F.Cu at (108.4, 95.3)
- C1, C3, C4, R5: moved to B.Cu
- C5, R4, U2: moved to F.Cu
- moved R4 20.0 mm to (101.6, 95.3), turned to 180 degrees
- moved C5 19.6 mm to (101.8, 93.5), turned to 180 degrees
- moved R7 16.8 mm to (107.4, 97.3), turned to 0 degrees
- moved R6 14.2 mm to (105.2, 95.4), turned to 0 degrees
- moved U2 12.1 mm to (103.9, 98.3), turned to 90 degrees
- moved Q1 10.2 mm to (108.9, 101.0), turned to 0 degrees
- moved R3 9.39 mm to (105.4, 102.0), turned to 90 degrees
- moved R5 9.12 mm to (108.9, 98.2), turned to 0 degrees
- moved L1 2.98 mm to (102.9, 99.3), turned to 90 degrees
- moved C4 2.67 mm to (94.2, 110.6), turned to 270 degrees
- moved C3 2.59 mm to (96.0, 110.7), turned to 270 degrees
- moved C1 2.27 mm to (95.0, 104.2), turned to 0 degrees
- moved D1 0.67 mm to (102.9, 92.6)
Routing:
- net +5V: track 123.9 -> 105.2 mm, vias 6 -> 4
- net +12V: track 161.6 -> 168.7 mm, vias 2 -> 3
- net R_GND: track 63.9 -> 68.3 mm
- net B_INT: track 16.5 -> 13.2 mm, vias 1 -> 0
- net Net-(R3-Pad2): track 0.00 -> 1.89 mm, vias 1 -> 0
- net Net-(C5-Pad1): track 6.62 -> 4.78 mm
- net Net-(C3-Pad1): track 0.00 -> 1.76 mm, vias 1 -> 0
- net +3.3V: track 5.92 -> 7.68 mm
- net Net-(Q1-Pad2): track 7.82 -> 8.92 mm
- net VFB: track 1.77 -> 2.28 mm, vias 1 -> 0
- net GND: track 40.4 -> 40.6 mm, vias 81 -> 110
- added copper zone on F.Cu, net VFB
Other:
- board text added: "v0.0.1 02/05/21"
- board text removed: "v0.0.0 01/23/21"

Commit message: Update to use MIC2250
Parts:
- removed the D1 at (102.9, 92.6)
- removed Q5: DMG2302U, Package_TO_SOT_SMD:SOT-23
- removed the R12 at (95.8, 93.0)
- removed the R15 at (91.8, 94.3)
- removed the R17 at (106.0, 92.7)
- removed the R7 at (107.4, 97.3)
- removed the R8 at (93.2, 102.5)
- removed the R9 at (86.4, 99.1)
- removed VFB: Test_Point_2.67x1.02mm, digikey-footprints:Test_Point_2.67x1.02mm
- added C7: 2.2uF_15v, Capacitor_SMD:C_0603_1608Metric, B.Cu at (93.0, 97.5)
- added C8: 10uF_6.3v, Capacitor_SMD:C_0603_1608Metric, B.Cu at (94.0, 83.0)
- added D40: D, Diode_SMD:D_SMA, B.Cu at (96.0, 94.0)
- added J1: Conn_01x03, Jumper:SolderJumper-3_P1.3mm_Open_Pad1.0x1.5mm_NumberLabels, B.Cu at (74.6, 75.0)
- added J2: Conn_01x03, Jumper:SolderJumper-3_P1.3mm_Open_Pad1.0x1.5mm_NumberLabels, B.Cu at (67.3, 113.5)
- added J3: Conn_01x03, Jumper:SolderJumper-3_P1.3mm_Open_Pad1.0x1.5mm_NumberLabels, B.Cu at (136.0, 93.1)
- added R21: 100R, Resistor_SMD:R_0805_2012Metric, F.Cu at (107.0, 101.5)
- added R23: 100R, Resistor_SMD:R_0805_2012Metric, F.Cu at (107.0, 97.5)
- added R24: 1MR, Resistor_SMD:R_0805_2012Metric, F.Cu at (112.0, 99.0)
- added R26: 1MR, Resistor_SMD:R_0805_2012Metric, F.Cu at (90.0, 100.7)
- added R27: 1MR, Resistor_SMD:R_0805_2012Metric, F.Cu at (100.0, 109.5)
- added R29: 10kR, Resistor_SMD:R_0805_2012Metric, B.Cu at (94.0, 85.0)
- added R30: 1MR, Resistor_SMD:R_0805_2012Metric, B.Cu at (91.0, 91.0)
- C2, C6: value 10uF -> 10kpF; footprint Capacitor_THT:CP_Radial_D4.0mm_P1.50mm -> Capacitor_SMD:C_0603_1608Metric
- C5: moved to B.Cu
- L1: value ASPI-8040S-620M -> 10uH; footprint Inductor_SMD:L_Taiyo-Yuden_NR-80xx -> Inductor_SMD:L_Taiyo-Yuden_NR-50xx
- Q1, R20: moved to F.Cu
- R1: value 10kR -> 1kR
- R2, R3: value 10kR -> 1kR; moved to B.Cu
- R22: value 1MR -> 100R
- R25: value 100R -> 1MR; moved to F.Cu
- R28: value 1MR -> 118kR; moved to B.Cu
- R4: value 100kR -> 10kR; moved to B.Cu
- R5: value 300R -> 10kR; moved to F.Cu
- R6: value 1.6MR -> 10kR; moved to B.Cu
- U1: value TC2014-3.3VxCTTR -> ATtiny461-20SU; footprint Package_TO_SOT_SMD:SOT-23-5 -> Package_SO:TSSOP-20_4.4x6.5mm_P0.65mm; moved to F.Cu
- U2: value MCP1640CH -> TC2014-3.3VxCTTR; footprint Package_TO_SOT_SMD:SOT-23-6 -> Package_TO_SOT_SMD:SOT-23-5; moved to B.Cu
- U3: value ATtiny13A-SSU -> MIC2250; footprint Package_SO:SOIC-8_3.9x4.9mm_P1.27mm -> Package_TO_SOT_SMD:TSOT-23-5
- X1: value SXO-53C3A071 -> SXO-53C
- moved C3 39.1 mm to (130.5, 92.4), turned to 90 degrees
- moved R1 37.9 mm to (77.6, 75.0)
- moved C2 35.8 mm to (72.8, 114.2), turned to 270 degrees
- moved C1 32.2 mm to (80.1, 75.7), turned to 270 degrees
- moved R3 29.0 mm to (133.0, 93.1), turned to 180 degrees
- moved R28 28.9 mm to (91.0, 87.5), turned to 90 degrees
- moved R2 27.7 mm to (70.3, 113.5), turned to 0 degrees
- moved REF** 24.5 mm to (109.7, 72.1)
- moved C6 23.9 mm to (90.5, 108.5), turned to 270 degrees
- moved Q3 23.2 mm to (87.0, 100.7), turned to 180 degrees
- moved R20 17.2 mm to (107.0, 95.5), turned to 0 degrees
- moved C5 16.6 mm to (96.4, 109.2), turned to 270 degrees
- moved R22 16.3 mm to (107.0, 99.5), turned to 0 degrees
- moved R4 15.8 mm to (99.5, 111.0), turned to 0 degrees
- moved R6 15.3 mm to (92.5, 103.9), turned to 90 degrees
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- renumbered D26 to D1, D20 to D10, D23 to D11, D27 to D12, D32 to D13, D37 to D14, D3 to D15, D6 to D16, D9 to D17, D12 to D18, D15 to D19, D31 to D2, D18 to D20, D24 to D22, D28 to D23, D33 to D24, D38 to D25, D4 to D26, D7 to D27, D10 to D28, D13 to D29, D36 to D3, D16 to D30, D19 to D31, D22 to D32, D25 to D33, D29 to D34, D34 to D35, D39 to D36, D30 to D37, D35 to D38, D40 to D39, D2 to D4, D8 to D6, D11 to D7, D14 to D8, D17 to D9, J2 to J4, J1 to J5, R13 to R12, R14 to R13, R16 to R14, R18 to R15, R19 to R16, R21 to R17, R23 to R18, R24 to R19, R26 to R7, R27 to R8, R29 to R9
Connections:
- C1 pad 1: +5V -> Hue
- C2 pad 1: +5V -> Sat
- C3 pad 1: Net-(C3-Pad1) -> Lum
- C4 pad 1: +3.3V -> Net-(C4-Pad1)
- C5 pad 1: Net-(C5-Pad1) -> +3.3V
- C6 pad 1: +12V -> GND
- C6 pad 2: GND -> +5V
- J4 pad 1: G -> MISO
- J4 pad 3: B -> SCK
- L1 pad 2: B_INT -> Net-(D40-Pad2)
- Q1 pad 1: +5V -> Net-(Q1-Pad1)
- Q1 pad 2: Net-(Q1-Pad2) -> GND
- Q1 pad 3: B_INT -> R_GND
- R1 pad 1: Net-(R1-Pad1) -> Net-(J1-Pad2)
- R1 pad 2: +3.3V -> Hue
- R2 pad 1: Net-(R2-Pad1) -> Net-(J2-Pad2)
- R2 pad 2: +5V -> Sat
- R20 pad 1: G -> R
- R20 pad 2: Net-(Q4-Pad1) -> Net-(Q1-Pad1)
- R22 pad 1: Net-(Q4-Pad1) -> B
- R22 pad 2: GND -> Net-(Q3-Pad1)
- R25 pad 1: MOSI -> Net-(Q2-Pad1)
- R25 pad 2: Net-(Q5-Pad1) -> GND
- R28 pad 1: Net-(Q5-Pad1) -> Net-(R28-Pad1)
- R3 pad 1: +5V -> Net-(J3-Pad2)
- R3 pad 2: Net-(R3-Pad2) -> Lum
- R4 pad 1: Net-(C5-Pad1) -> Net-(R4-Pad1)
- R4 pad 2: GND -> +3.3V
- R5 pad 1: Net-(Q1-Pad2) -> RESET
- R5 pad 2: B_INT -> +5V
- R6 pad 1: +12V -> Net-(R6-Pad1)
- R6 pad 2: VFB -> +5V
- U1 pad 1: +5V -> MOSI
- U1 pad 2: GND -> MISO
- U1 pad 3: Net-(R2-Pad1) -> SCK
- U1 pad 4: Net-(C3-Pad1) -> (no net)
- U1 pad 5: +3.3V -> +5V
- U2 pad 1: Net-(Q1-Pad2) -> +5V
- U2 pad 3: Net-(R3-Pad2) -> Net-(R6-Pad1)
- U2 pad 4: VFB -> Net-(C4-Pad1)
- U2 pad 5: Net-(C5-Pad1) -> +3.3V
- U3 pad 1: RESET -> Net-(D40-Pad2)
- U3 pad 2: 20MHZ -> GND
- U3 pad 3: W -> Net-(R28-Pad1)
- U3 pad 4: GND -> Net-(R29-Pad1)
- U3 pad 5: MOSI -> +5V
- X1 pad 1: Net-(R1-Pad1) -> Net-(R4-Pad1)
- X1 pad 3: 20MHZ -> CLK
Routing:
- net +5V: track 105.2 -> 184.3 mm, vias 4 -> 8
- net Hue: track 0.00 -> 68.0 mm, vias 0 -> 3
- net Sat: track 0.00 -> 45.2 mm, vias 0 -> 3
- net Net-(Q5-Pad1): track 44.5 -> 0.00 mm, vias 3 -> 0
- net Lum: track 0.00 -> 40.7 mm, vias 0 -> 3
- net B: track 41.1 -> 3.17 mm, vias 4 -> 0
- net SCK: track 0.00 -> 36.1 mm, vias 0 -> 1
- net W_GND: track 96.5 -> 132.0 mm, vias 6 -> 3
- net MISO: track 0.00 -> 32.6 mm, vias 0 -> 1
- net G: track 31.7 -> 2.79 mm, vias 4 -> 0
- net B_GND: track 100.5 -> 118.7 mm
- net G_GND: track 92.7 -> 106.9 mm, vias 8 -> 3
- net GND: track 40.6 -> 54.3 mm, vias 110 -> 45
- net B_INT: track 13.2 -> 0.00 mm
- net Net-(Q4-Pad1): track 29.8 -> 18.7 mm, vias 1 -> 0
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- removed copper zone on F.Cu, net VFB
Other:
- board text added: "Hue"
- board text added: "Luminosity"
- board text added: "Saturation"
- board text added: "v1.0.0 06/14/21"
- board text removed: "v0.0.1 02/05/21"
